Commit message: Full system update: Integrated Vision-Based Goal Navigation

File: urdf/robot.urdf (robot description, URDF)
Before this commit: robot diff_drive_robot, 7 links, 6 joints
Links:
- added link base_footprint
- added link camera_link; collision box size=0.015 0.08 0.022; visual box size=0.015 0.08 0.022
- added link camera_link_optical
Joints:
- added joint base_footprint_joint: type fixed, parent base_footprint, child base_link, origin xyz=0 0 0 rpy=0 0 0
- added joint camera_joint: type fixed, parent chassis, child camera_link, origin xyz=0.28 0 0.08 rpy=0 0 0
- added joint camera_optical_joint: type fixed, parent camera_link, child camera_link_optical, origin xyz=0 0 0 rpy=${-pi/2} 0 ${-pi/2}
